File: Hardware/JBT01.kicad_sch (KiCad schematic)
At the start: 79 parts, among them CN1 Conn_01x01_Male, CN10 Conn_01x01_Male, CN11 Conn_01x01_Male, CN12 Conn_01x01_Male, CN13 Conn_01x01_Male, CN14 Conn_01x01_Male, CN15 Conn_01x01_Male, CN16 Conn_01x01_Male, CN2 Conn_01x01_Male, CN3 Conn_01x01_Male, CN4 Conn_01x01_Male, CN5 Conn_01x01_Male, CN6 Conn_01x01_Male, CN7 Conn_01x01_Male, CN8 Conn_01x01_Male, CN9 Conn_01x01_Male, J1 Conn_01x02, J10 Conn_01x16, J11 Conn_01x02, J2 Conn_01x02, J3 Screw_Terminal_01x02, J4 Conn_01x02, J5 Conn_01x02, J6 Screw_Terminal_01x02, J7 Conn_01x05, J8 Conn_01x05, J9 Conn_01x02, K1 RELAY-T91-30A, Q1 MMBT2222A, SW1 RED, SW2 GREEN, U1 MS51FB9AE, U2 EL817, U3 AMS1117-5V, U4 MAX6675

Commit message: Update KiCad files of Rev C and enhance schematic title block
Other:
- title: (none) -> JBT01
Changed lines of the file:
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@@
 (kicad_sch (version 20211123) (generator eeschema)
   (paper "A4")
+  (title_block
+    (title "JBT01")
+    (date "29-04-2023")
+    (rev "C")
+  )
   (junction (at 38.735 67.31) (diameter 0) (color 0 0 0 0)
   )
